File: hardware/kicad/MC6800/MC6800.kicad_sch (KiCad schematic)
At the start: 43 parts, among them J1 SD_Card_Receptacle, J2 DIN41612_02x32_AB, U1 MC68B00, U10 74LS670, U11 74LS670, U12 74LS670, U13 AS6C4008-55PCN, U14 HM628128D_DIP32_SOP32, U15 74LS244, U16 AS6C1008-xxP, U17 74LS245, U18 74LS245, U19 74LS245, U2 MC68B21, U20 74LS245, U21 74LS166, U22 74HCT164, U23 74LS573, U24 74LS574, U25 74LS299, U26 74LS163, U27 74LS174, U28 74LS174, U29 74LS00, U3 MC68B50, U30 74LS02, U31 74LS138, U32 74LS153, U33 74LS157, U34 74LS139, U35 74LS165, U36 74LS175, U37 74LS191, U38 74LS190, U39 74LS193, U4 MC68B50, U5 MC68B40, U6 MC68B44, U7 28C256, U8 HM62256BLP, U9 74LS670, Y1 CXO_DIP8, Y2 CXO_DIP8

Commit message: 20260210
Parts:
- added C1, C2, C3, C4, C5, C6, C7: 100nF, symbol Device:C
- added U40, U49: KM28C64A, Package_DIP:DIP-28_W15.24mm, symbol Memory_EEPROM:KM28C64A
- added U41, U42: MAX232, symbol Interface_UART:MAX232
- added U43: 74LS00, symbol 74xx:74LS00
- added U44, U45: 74LS04, symbol 74xx:74LS04
- added U46: MC68B03, Package_DIP:DIP-40_W15.24mm, symbol MC6800:MC68B03
- added U47, U58: 74LS573, symbol 74xx:74LS573
- added U48: 74LS245, symbol 74xx:74LS245
- added U50, U51: 74LS670, symbol 74xx:74LS670
- added U52: AS6C4008-55PCN, Package_DIP:DIP-32_W15.24mm, symbol Memory_RAM:AS6C4008-55PCN
- added U53: MC68B40, Package_DIP:DIP-28_W15.24mm, symbol Interface:MC68B40
- added U54: MC68B50, Package_DIP:DIP-24_W15.24mm, symbol Interface_UART:MC68B50
- added U55: HM62256BLP, Package_DIP:DIP-28_W15.24mm, symbol Memory_RAM:HM62256BLP
- added U56: MC68B21, Package_DIP:DIP-40_W15.24mm, symbol Interface:MC68B21
- added U57: MC146818, Package_DIP:DIP-24_W15.24mm, symbol MC6800:MC146818
- added U59: 74LS74, symbol 74xx:74LS74
- added U60, U61: 74LS02, symbol 74xx:74LS02
- added U62: MC68B44, Package_DIP:DIP-40_W15.24mm, symbol Interface:MC68B44
- added U63: 6264, Package_DIP:DIP-28_W7.62mm, symbol MC6800:6264
- added Y4: CXO_DIP8, Oscillator:Oscillator_DIP-8, symbol MC6800:CXO_DIP8
Connections:
- net GND: now reaches Y1.4 (GND)
- net GND: now also C1.2, C2.2, C3.2, C4.2, C5.2, C6.2, C7.2, U46.1 (VSS), U47.10 (GND), U48.10 (GND), U50.8 (GND), U51.8 (GND), U58.1 (OE), U58.10 (GND), U63.14 (GND)
- net at Y1.5 (OUT): now also U43.1, U44.1
- net VDD: now reaches Y1.8 (Vcc)
- net VDD: now also C1.1, C2.1, C3.1, C4.1, C5.1, C6.1, C7.1, U46.21 (VCCSTBY), U46.7 (VCC), U47.20 (VCC), U50.16 (VCC), U51.16 (VCC), U58.20 (VCC), U63.28 (V_{CC})
- new net: U60.10, U63.3 (A_{7})
- new net: U43.3, U43.4, U45.3
- new net: U43.5, U44.2
- new net: U43.2, U43.6, U45.5
- new net: U61.13, U63.2 (A_{12})
- new net: U61.4, U63.21 (A_{10})
- new net: U61.1, U63.24 (A_{9})
- new net: U61.10, U63.23 (A_{11})
- new net: U60.13, U63.25 (A_{8})
- new net: U60.1, U63.5 (A_{5})
- new net: U60.4, U63.4 (A_{6})
- new net A0: U47.19 (Q0), U50.14 (Wa), U51.14 (Wa)
- new net A1: U47.18 (Q1), U50.13 (Wb), U51.13 (Wb)
- new net A10: U46.27 (A10)
- new net A11: U46.26 (A11)
- new net A12: U46.25 (A12)
- new net A13: U46.24 (A13)
- new net A14: U46.23 (A14), U50.10 (Q1)
- new net A15: U46.22 (A15), U50.9 (Q2)
- new net A16: U50.7 (Q3)
- new net A17: U50.6 (Q4)
- new net A18: U51.10 (Q1)
- new net A19: U51.9 (Q2)
- new net A2: U47.17 (Q2)
- new net A20: U51.7 (Q3)
- new net A21: U51.6 (Q4)
- new net A3: U47.16 (Q3)
- new net A4: U47.15 (Q4)
- new net A5: U47.14 (Q5)
- new net A6: U47.13 (Q6)
- new net A7: U47.12 (Q7)
- new net A8: U46.29 (A8)
- new net A9: U46.28 (A9)
- new net AD0: U46.37 (AD0), U47.2 (D0), U48.2 (A0)
- new net AD1: U46.36 (AD1), U47.3 (D1), U48.3 (A1)
- new net AD2: U46.35 (AD2), U47.4 (D2), U48.4 (A2)
- new net AD3: U46.34 (AD3), U47.5 (D3), U48.5 (A3)
- new net AD4: U46.33 (AD4), U47.6 (D4), U48.6 (A4)
- new net AD5: U46.32 (AD5), U47.7 (D5), U48.7 (A5)
- new net AD6: U46.31 (AD6), U47.8 (D6), U48.8 (A6)
- new net AD7: U46.30 (AD7), U47.9 (D7), U48.9 (A7)
- new net AS: U46.39 (AS), U47.11 (Load)
- new net CLK: U59.3 (C)
- new net D0: U48.18 (B0), U50.15 (D1), U58.2 (D0)
- new net D1: U48.17 (B1), U50.1 (D2), U58.3 (D1)
- new net D2: U48.16 (B2), U50.2 (D3), U58.4 (D2)
- new net D3: U48.15 (B3), U50.3 (D4), U58.5 (D3)
- new net D4: U48.14 (B4), U51.15 (D1), U58.6 (D4)
- new net D5: U48.13 (B5), U51.1 (D2), U58.7 (D5)
- new net D6: U48.12 (B6), U51.2 (D3), U58.8 (D6)
- new net D7: U48.11 (B7), U51.3 (D4), U58.9 (D7)
- new net E: U46.40 (E)
- new net PID0: U58.19 (Q0), U60.3
- new net PID1: U58.18 (Q1), U60.6
- new net PID2: U58.17 (Q2), U60.9
- new net PID3: U58.16 (Q3), U60.12
- new net PID4: U58.15 (Q4), U61.3
- new net PID5: U58.14 (Q5), U61.6
- new net PID6: U58.13 (Q6), U61.9
- new net PID7: U58.12 (Q7), U61.12
- new net Phi1: U45.6
- new net Phi2: U45.4
- new net R/~{W}: U46.38 (R/~{W})
- new net SUP/~{USER}: U59.5 (Q), U60.11, U60.2, U60.5, U60.8, U61.11, U61.2, U61.5, U61.8
- new net VA13: U63.10 (A_{0})
- new net VA14: U50.5 (Ra), U51.5 (Ra), U63.9 (A_{1})
- new net VA15: U50.4 (Rb), U51.4 (Rb), U63.8 (A_{2})
- new net ~{RESET}: U59.4 (~{S})
- no-connect marks 0 -> 1
Other:
- note added: "Componenets to add: ------------------- Floppy controller. FPU. To do: ------ Memory map, address decoding. SPI MMDS like debug/trace. DMA cycles when E is low? A14-A21 generation during DMA. Slow peripheral bus (RTC). Mode entry following reset."
- note added: "Swtich to Supervisor mode: -------------------------- 1-Fetch byte in the vector area && A15 == 0; => State = 1; else State = 0; 2-Immediatelly fetch byte in the vector area + 1 && State == 1; => State = 2; else State = 0; 3-Immediately fetch opcode in designated OS range && State == 2; => Mode = Supervisor; State = 0; What to do if an NMI is triggered while in the vector fetch sequence? OS Range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"
- note added: "Things MMU Needs to do: ----------------------- -Reset: after reset MMU should allow CPU to access vector area in ROM and initialize MMU. -On an interrupt of SWI OS may need access to USER stack. First to save but also for contents. -Switch to OS/Supervisor mode in case of SWI, interrupts, NMI. -Sequence to switch back to user mode. User Process: ------------- 0x0000-0xMFFF Data page (Can be set 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"
- moved on the sheet: J1, U13, U14, U16, U2, U21, U22, U23, U24, U25, U26, U27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
